File: power.kicad_sch (KiCad schematic)
At the start: 15 parts, among them J4 Conn_01x02_Socket, Q1 JSM2302, SW1 On/Off, U5 TP4057, U7 DS8242-33S3

Commit message: Fix footprint bugs (and remove WS2811 interfaces).  Part of #5
Parts:
- J4: footprint Connector_JST:JST_PH_B2B-PH-SM4-TB_1x02-1MP_P2.00mm_Vertical -> Connector_JST:JST_PH_S2B-PH-SM4-TB_1x02-1MP_P2.00mm_Horizontal
Changed lines of the file:
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@@
 			)
 		)
-		(property "Footprint" "Connector_JST:JST_PH_B2B-PH-SM4-TB_1x02-1MP_P2.00mm_Vertical"
+		(property "Footprint" "Connector_JST:JST_PH_S2B-PH-SM4-TB_1x02-1MP_P2.00mm_Horizontal"
 			(at 137.16 57.15 0)
 			(effects
